Commit message: modify the rover gazebo model and realize two uav landing on a rover simulation

File: uavros_simulation/uavros_gazebo/models/rover/rover.urdf (robot description, URDF)
Before this commit: robot rover, 2 links, 1 joints
Links:
- added link front_left_wheel
- added link front_right_wheel
- added link front_right_wheel_steering_block
- added link rear_left_wheel
- added link rear_right_wheel
Joints:
- added joint front_left_wheel_joint: type continuous, parent front_left_wheel_steering_block, child front_left_wheel, limit effort=10000.0 velocity=100.0
- added joint front_right_steering_joint: type revolute, parent base_link, child front_right_wheel_steering_block, limit lower=-0.7727 upper=0.7727 effort=1000.0 velocity=100.0
- added joint front_right_wheel_joint: type continuous, parent front_right_wheel_steering_block, child front_right_wheel, limit effort=10000.0 velocity=100.0
- added joint rear_left_wheel_joint: type continuous, parent base_link, child rear_left_wheel, limit effort=10000.0 velocity=100.0
- added joint rear_right_wheel_joint: type continuous, parent base_link, child rear_right_wheel, limit effort=10000.0 velocity=100.0
- joint front_left_steering_joint: axis 0 0 1 -> (none); origin xyz=1.20222 0.5 0.35515 rpy=1.57079 0 0 -> (none)
